File: resources/sample/blinker-555.kicad_pcb (KiCad board)
At the start: 2 copper layers, 60 x 45 mm, 7 parts, among them U1 NE555

Commit message: fix(live-bench): LED polarity — coach follows the resolved pinMap; fix blinker-555 board
The dark-LED coach assumed pad 1 = anode, but the deck generator wires
diodes by the resolved pinMap, and the bundled library LED_* entries
follow the KiCad convention (pad 1 = cathode) — so the coach polarity
verdict was inverted relative to what was actually simulated.
buildCoachInput now derives each LED's anode/cathode pads from the
part's resolved pinMap (SPICE diode position 1 = anode), falling back
to the KiCad convention when a part has no pinMap. The coach and the
sim can no longer disagree.

blinker-555.kicad_pcb had the same reversed LED first-light shipped
with (pad1=LED_A, pad2=GND -> reverse-biased, dark) — swapped, so the
555 demo LED actually blinks now that the live transient glow drives
it. New sample-board guard pins D1 pad1=GND / pad2=drive-net on BOTH
bundled boards so a reversed demo LED can never ship again.

Suite: 1071 passed, typecheck clean.

Co-Authored-By: Claude Fable 5 <noreply@anthropic.com>
Connections:
- D1 pad 1: LED_A -> GND
- D1 pad 2: GND -> LED_A
Changed lines of the file:
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@@
       (effects (font (size 1 1) (thickness 0.15))))
     (pad "1" smd roundrect (at -0.9125 0) (size 1.025 1.4)
+      (layers "F.Cu" "F.Paste" "F.Mask") (roundrect_rratio 0.25) (net 2 "GND"))
+    (pad "2" smd roundrect (at 0.9125 0) (size 1.025 1.4)
       (layers "F.Cu" "F.Paste" "F.Mask") (roundrect_rratio 0.25) (net 6 "LED_A"))
-    (pad "2" smd roundrect (at 0.9125 0) (size 1.025 1.4)
-      (layers "F.Cu" "F.Paste" "F.Mask") (roundrect_rratio 0.25) (net 2 "GND"))
   )
   (segment (start 15.9125 12) (end 25 12) (width 0.25) (layer "F.Cu") (net 3 "DISCH"))
